File: sama5d27_som1_ek-sharp_ls0xx_lcd-adapter.kicad_pcb (KiCad board)
At the start: 2 copper layers, 50.1 x 80.2 mm, 14 parts, among them J1 XF2M-5015-1A, J2 1-1734592-0

Commit message: Pump to revision A1 (replacing J2)
Parts:
- J2: value 1-1734592-0 -> 51441-1093; footprint footprints:1-1734592-0 -> footprints:51441-1093
- moved J2 2.88 mm to (186.2, 99.0)
Connections:
- J2 pad 1: GND -> /SPI0_SPCK_SCK
- J2 pad 10: /SPI0_SPCK_SCK -> GND
- J2 pad 2: GND -> /SPI0_MOSI_SI
- J2 pad 3: /EXTMODE -> /SPI0_NPCS0_SCS
- J2 pad 4: +5V -> /EXTCOMIN
- J2 pad 5: +5V -> /LCD_DISP_DISP
- J2 pad 6: /LCD_DISP_DISP -> +5V
- J2 pad 7: /EXTCOMIN -> +5V
- J2 pad 8: /SPI0_NPCS0_SCS -> /EXTMODE
- J2 pad 9: /SPI0_MOSI_SI -> GND
Routing:
- net /SPI0_SPCK_SCK: track 94.1 -> 96.4 mm
- net /SPI0_MOSI_SI: track 92.8 -> 94.5 mm
- net GND: track 79.5 -> 80.9 mm, vias 5 -> 6
- net /EXTCOMIN: track 30.3 -> 28.9 mm
- net /SPI0_NPCS0_SCS: track 91.2 -> 89.8 mm
- net /LCD_DISP_DISP: track 73.0 -> 72.4 mm

Commit message: Update RevA1
Parts:
- moved REF** 3.75 mm to (211.5, 22.5)
- moved REF** 3.61 mm to (163.5, 22.5)
- moved REF** 2.46 mm to (211.5, 100.5)
- moved REF** 2.24 mm to (163.5, 100.5)
- moved J1 2.05 mm to (187.4, 24.5)
Routing:
- net GND: track 80.9 -> 85.9 mm
- net /LCD_PWM: track 60.4 -> 62.5 mm
- net /5V: track 64.8 -> 66.8 mm
- net /SPI0_SPCK_SCK: track 96.4 -> 98.2 mm
- net /SPI0_NPCS0_SCS: track 89.8 -> 91.6 mm
- net /SPI0_MOSI_SI: track 94.5 -> 96.3 mm
- net /LCD_DISP_DISP: track 72.4 -> 74.2 mm
Other:
- board size 50.1 x 80.2 mm -> 55 x 85 mm
- board text added: "J1"
- board text added: "J2"

Commit message: Centralize pcb in sheet
Parts:
- moved R2 51.7 mm to (146.8, 128.0)
- moved R3 51.7 mm to (150.4, 128.0)
- moved R1 51.7 mm to (145.2, 122.9)
- moved R5 51.7 mm to (148.6, 119.7)
- moved REF** 51.7 mm to (123.8, 55.6)
- moved REF** 51.7 mm to (123.8, 133.6)
- moved C1 51.7 mm to (145.0, 125.2)
- moved C2 51.7 mm to (148.7, 122.9)
- moved C3 51.7 mm to (148.7, 125.0)
- moved J1 51.7 mm to (147.7, 57.6)
- moved J2 51.7 mm to (146.5, 132.2)
- moved REF** 51.7 mm to (171.8, 55.6)
- moved R4 51.7 mm to (145.2, 119.7)
- moved REF** 51.7 mm to (171.8, 133.6)

Commit message: Update revision text on board
Other:
- board text added: "Sharp memory LCD Breakout Rev. A1"
- board text removed: "Sharp memory LCD Breakout Rev. A0"
